Commit message: Updates for Gazebo fidelity and moveit-servo control

File: panda_description/urdf/panda_xacro/hand.xacro (robot description, xacro)
@@ -2,5 +2,6 @@
 <robot xmlns:xacro="http://www.ros.org/wiki/xacro" name="hand">
   <!-- Gazebo adaptation: dynamics (dampening)-->
-  <xacro:property name="joint_damping" value="1.0"/>
+  <xacro:property name="joint_damping" value="5.0"/>
+  <xacro:property name="gripper_joint_friction" value="100.0"/>
   <!-- END Gazebo adaptation-->
   <xacro:macro name="hand" params="description_pkg:='panda' connected_to:='' ns:='' rpy:='0 0 0' xyz:='0 0 0' ">
@@ -79,7 +80,7 @@
       <origin xyz="0 0 0.0584" rpy="0 0 0"/>
       <axis xyz="0 1 0"/>
-      <limit effort="20" lower="0.0" upper="0.04" velocity="0.2"/>
+      <limit effort="100" lower="0.0" upper="0.04" velocity="0.2"/>
       <!-- Gazebo adaptation: dampening-->
-      <dynamics damping="${joint_damping}"/>
+      <dynamics damping="${joint_damping}" friction="${gripper_joint_friction}"/>
       <!-- END Gazebo adaptation-->
     </joint>
@@ -89,7 +90,7 @@
       <origin xyz="0 0 0.0584" rpy="0 0 0"/>
       <axis xyz="0 -1 0"/>
-      <limit effort="20" lower="0.0" upper="0.04" velocity="0.2"/>
+      <limit effort="100" lower="0.0" upper="0.04" velocity="0.2"/>
       <!-- Gazebo adaptation: dampening-->
-      <dynamics damping="${joint_damping}"/>
+      <dynamics damping="${joint_damping}" friction="${gripper_joint_friction}"/>
       <!-- END Gazebo adaptation-->
     </joint>

File: panda_description/urdf/panda_xacro/panda.gazebo.xacro (robot description, xacro)
@@ -2,4 +2,48 @@
 <robot xmlns:xacro="http://www.ros.org/wiki/xacro">
     <xacro:macro name="panda_gazebo" params="robot_name">
+        <!-- finger_joint1 -->
+        <gazebo reference="${robot_name}_finger_joint1">
+            <implicitSpringDamper>1</implicitSpringDamper>
+        </gazebo>
+        <!-- finger_joint2 -->
+        <gazebo reference="${robot_name}_finger_joint2">
+            <implicitSpringDamper>1</implicitSpringDamper>
+        </gazebo>
+        <!-- joint0 -->
+        <gazebo reference="${robot_name}_joint0">
+            <implicitSpringDamper>1</implicitSpringDamper>
+        </gazebo>
+        <!-- joint1 -->
+        <gazebo reference="${robot_name}_joint1">
+            <implicitSpringDamper>1</implicitSpringDamper>
+        </gazebo>
+        <!-- joint2 -->
+        <gazebo reference="${robot_name}_joint2">
+            <implicitSpringDamper>1</implicitSpringDamper>
+        </gazebo>
+        <!-- joint3 -->
+        <gazebo reference="${robot_name}_joint3">
+            <implicitSpringDamper>1</implicitSpringDamper>
+        </gazebo>
+        <!-- joint4 -->
+        <gazebo reference="${robot_name}_joint4">
+            <implicitSpringDamper>1</implicitSpringDamper>
+        </gazebo>
+        <!-- joint5 -->
+        <gazebo reference="${robot_name}_joint5">
+            <implicitSpringDamper>1</implicitSpringDamper>
+        </gazebo>
+        <!-- joint6 -->
+        <gazebo reference="${robot_name}_joint6">
+            <implicitSpringDamper>1</implicitSpringDamper>
+        </gazebo>
+        <!-- joint7 -->
+        <gazebo reference="${robot_name}_joint7">
+            <implicitSpringDamper>1</implicitSpringDamper>
+        </gazebo>
+        <!-- joint8 -->
+        <gazebo reference="${robot_name}_joint8">
+            <implicitSpringDamper>1</implicitSpringDamper>
+        </gazebo>
         <!-- Link0 -->
         <gazebo reference="${robot_name}_link0">
@@ -7,4 +51,6 @@
             <mu1>0.2</mu1>
             <mu2>0.2</mu2>
+            <turnGravityOff>true</turnGravityOff>
+            <!-- gravity is turned off in all these links because moveit_servo + roscontrol don't have gravity compensation built in. -->
         </gazebo>
         <!-- Link1 -->
@@ -13,4 +59,5 @@
             <mu1>0.2</mu1>
             <mu2>0.2</mu2>
+            <turnGravityOff>true</turnGravityOff>
         </gazebo>
         <!-- Link2 -->
@@ -19,4 +66,5 @@
             <mu1>0.2</mu1>
             <mu2>0.2</mu2>
+             <turnGravityOff>true</turnGravityOff>
         </gazebo>
         <!-- Link3 -->
@@ -25,4 +73,5 @@
             <mu1>0.2</mu1>
             <mu2>0.2</mu2>
+             <turnGravityOff>true</turnGravityOff>
         </gazebo>
         <!-- Link4 -->
@@ -31,4 +80,5 @@
             <mu1>0.2</mu1>
             <mu2>0.2</mu2>
+             <turnGravityOff>true</turnGravityOff>
         </gazebo>
         <!-- Link5 -->
@@ -37,4 +87,5 @@
             <mu1>0.2</mu1>
             <mu2>0.2</mu2>
+             <turnGravityOff>true</turnGravityOff>
         </gazebo>
         <!-- Link6 -->
@@ -43,4 +94,5 @@
             <mu1>0.2</mu1>
             <mu2>0.2</mu2>
+             <turnGravityOff>true</turnGravityOff>
         </gazebo>
         <!-- Link7 -->
@@ -49,4 +101,5 @@
             <mu1>0.2</mu1>
             <mu2>0.2</mu2>
+             <turnGravityOff>true</turnGravityOff>
         </gazebo>
         <!-- Link8 -->
@@ -55,4 +108,5 @@
             <mu1>0.2</mu1>
             <mu2>0.2</mu2>
+             <turnGravityOff>true</turnGravityOff>
         </gazebo>
         <!-- LinkHand -->
@@ -61,16 +115,63 @@
             <mu1>0.2</mu1>
             <mu2>0.2</mu2>
+            <turnGravityOff>true</turnGravityOff>
         </gazebo>
         <!-- LinkRightFinger -->
         <gazebo reference="${robot_name}_rightfinger">
+            <implicitSpringDamper>1</implicitSpringDamper>
             <material>Gazebo/Grey</material>
-            <mu1>0.2</mu1>
-            <mu2>0.2</mu2>
+            <mu1>5.0</mu1>
+            <mu2>5.0</mu2>
+            # from https://github.com/frankaemika/franka_ros/blob/develop/franka_description/robots/panda_gazebo.xacro
+            <kp>1e6</kp>
+            <kd>1e2</kd>
+            <minDepth>0.0</minDepth>
+            <maxVel>0.0</maxVel>
+            <torsional>
+                <ode>
+                    <coefficient>1000</coefficient>
+                    <slip>0</slip>
+                </ode>
+            </torsional>
+            <physics>
+                <max_contacts>20</max_contacts>
+                <ode>
+                <limit>
+                    <cfm>0</cfm>
+                    <erp>0.2</erp>
+                </limit>
+                <implicit_spring_damper>1</implicit_spring_damper>
+                </ode>
+            </physics>
+            <turnGravityOff>true</turnGravityOff>
         </gazebo>
         <!-- LinkLeftFinger -->
         <gazebo reference="${robot_name}_leftfinger">
             <material>Gazebo/Grey</material>
-            <mu1>0.2</mu1>
-            <mu2>0.2</mu2>
+            <implicitSpringDamper>1</implicitSpringDamper>
+            <mu1>5.0</mu1>
+            <mu2>5.0</mu2>
+            # from https://github.com/frankaemika/franka_ros/blob/develop/franka_description/robots/panda_gazebo.xacro
+            <kp>1e6</kp>
+            <kd>1e2</kd>
+            <minDepth>0.0</minDepth>
+            <maxVel>0.0</maxVel>
+            <torsional>
+                <ode>
+                    <coefficient>1000</coefficient>
+                    <slip>0</slip>
+                </ode>
+            </torsional>
+            <physics>
+                <max_contacts>20</max_contacts>
+                <ode>
+                <limit>
+                    <cfm>0</cfm>
+                    <erp>0.2</erp>
+                </limit>
+                <implicit_spring_damper>1</implicit_spring_damper>
+                </ode>
+            </physics>
+            <turnGravityOff>true</turnGravityOff>
         </gazebo>
     </xacro:macro>

File: panda_description/urdf/panda_xacro/panda_arm.xacro (robot description, xacro)
@@ -4,5 +4,7 @@
   <xacro:property name="joint_damping" value="1.0"/>
   <!-- END Gazebo adaptation-->
-  <xacro:macro name="panda_arm" params="arm_id:='panda' description_pkg:='panda_description' connected_to:='' xyz:='0 0 0' rpy:='0 0 0'">
+  <xacro:arg name="xyz" default="0 0 0" />
+  <xacro:arg name="rpy" default="0 0 0" />
+  <xacro:macro name="panda_arm" params="arm_id:='panda' description_pkg:='panda_description' connected_to:=''">
     <!-- Gazebo adaptation: Attach Robot rigidly to the world frame in Gazebo -->
     <link name="world" />
@@ -10,5 +12,5 @@
       <parent link="world" />
       <child link="${arm_id}_link0" />
-      <origin xyz="0.0 0.0 0.0" rpy="0.0 0.0 0.0" />
+      <origin xyz="$(arg xyz)" rpy="$(arg rpy)" />
       <!-- Gazebo adaptation: dampening-->
       <dynamics damping="${joint_damping}"/>

File: panda_description/urdf/panda_xacro/panda_arm_hand.urdf.xacro (robot description, xacro)
@@ -6,5 +6,6 @@
   <xacro:include filename="panda.transmission.xacro" />
   <xacro:panda_arm description_pkg="panda_description" />
-  <xacro:hand ns="panda" rpy="0 0 ${-pi/4}" connected_to="panda_link8" description_pkg="panda_description"/>
+  <!-- <xacro:hand ns="panda" rpy="0 0 ${-pi/4}" connected_to="panda_link8" description_pkg="panda_description"/> -->
+  <xacro:hand ns="panda" rpy="0 0 0" connected_to="panda_link8" description_pkg="panda_description"/>
   <xacro:panda_gazebo robot_name="panda" />
   <xacro:panda_transmission robot_name="panda" />
