Commit message: Working gazebo config

File: panda_description/urdf/panda_xacro/panda_arm.xacro (robot description, xacro)
@@ -72,5 +72,5 @@
       <child link="${arm_id}_link1"/>
       <axis xyz="0 0 1"/>
-      <limit effort="87" lower="-2.8973" upper="2.8973" velocity="2.1750"/>
+      <limit effort="870" lower="-2.8973" upper="2.8973" velocity="2.1750"/>
       <!-- Gazebo adaptation: dampening-->
       <dynamics damping="${joint_damping}"/>
@@ -102,5 +102,5 @@
       <child link="${arm_id}_link2"/>
       <axis xyz="0 0 1"/>
-      <limit effort="87" lower="-1.7628" upper="1.7628" velocity="2.1750"/>
+      <limit effort="870" lower="-1.7628" upper="1.7628" velocity="2.1750"/>
       <!-- Gazebo adaptation: dampening-->
       <dynamics damping="${joint_damping}"/>
@@ -132,5 +132,5 @@
       <child link="${arm_id}_link3"/>
       <axis xyz="0 0 1"/>
-      <limit effort="87" lower="-2.8973" upper="2.8973" velocity="2.1750"/>
+      <limit effort="870" lower="-2.8973" upper="2.8973" velocity="2.1750"/>
       <!-- Gazebo adaptation: dampening-->
       <dynamics damping="${joint_damping}"/>
@@ -162,5 +162,5 @@
       <child link="${arm_id}_link4"/>
       <axis xyz="0 0 1"/>
-      <limit effort="87" lower="-3.0718" upper="-0.0698" velocity="2.1750"/>
+      <limit effort="870" lower="-3.0718" upper="-0.0698" velocity="2.1750"/>
       <!-- Gazebo adaptation: dampening-->
       <dynamics damping="${joint_damping}"/>
